Commit message: changed inertial values, might need to change back if too unrealistic

File: aruco_model_generation/urdf/aruco_76.75mm/aruco_76.75mm_1.urdf (robot description, URDF)
Before this commit: robot rviz_test_name, 1 links, 0 joints
Links:
- link base_link: mass 1 -> 0.01

File: aruco_model_generation/urdf/common/base_aruco_panel.urdf.xacro (robot description, xacro)
@@ -33,7 +33,7 @@
         <mass value="1"/>
         <inertia
-            ixx="1.0" ixy="0.0" ixz="0.0"
-            iyy="1.0" iyz="0.0"
-            izz="1.0"/>
+            ixx="0" ixy="0.0" ixz="0.0"
+            iyy="0" iyz="0.0"
+            izz="0"/>
         </inertial>
     </link>
